File: d2tsf-hw.kicad_pcb (KiCad board)
At the start: 2 copper layers, 160.2 x 69.8 mm, 59 parts, among them J1 Reset MCU, J10 Serial, J11 Barrel_Jack_Switch, J12 Power, J13 RX In, J14 GND, J15 TX Out, J16 Port B, J2 Programming, J3 SHIFT0, J4 SHIFT1, J5 PSS, J6 1MHZ, J7 Reset F9T, J8 ANT_VCC, J9 F9T Connector, U1 AMS1117, U2 STM32F411RETx, U3 SN74LVC8T245PWR, U4 SN74LVC8T245PWR, U5 MAX3232, Y1 16MHz

Commit message: Change to use 4 layers
- In1 is GND layer
- In2 is 3.3V layer
- Additionally, a few test points were added
Parts:
- added C31: 1u, Capacitor_SMD:C_1210_3225Metric, F.Cu at (209.1, 75.1)
- added FB1: 33uH, Capacitor_SMD:C_0805_2012Metric, F.Cu at (212.7, 73.6)
- added TP1: SHIFT0, TestPoint:TestPoint_Pad_D1.0mm, F.Cu at (164.3, 105.1)
- added TP2: SHIFT1, TestPoint:TestPoint_Pad_D1.0mm, F.Cu at (169.6, 107.9)
- added TP3: PPS, TestPoint:TestPoint_Pad_D1.0mm, F.Cu at (194.3, 102.3)
- added TP4: 1MHZ, TestPoint:TestPoint_Pad_D1.0mm, F.Cu at (200.8, 104.9)
- C11: value 10p -> 10n
- J16: value Port B -> Conn_01x09_Male; footprint Connector_PinHeader_2.54mm:PinHeader_1x08_P2.54mm_Vertical -> Connector_PinHeader_2.54mm:PinHeader_1x09_P2.54mm_Vertical
- moved J8 12.4 mm to (204.4, 73.6)
- moved C30 10.6 mm to (115.1, 101.3), turned to 90 degrees
- moved C1 7.21 mm to (216.3, 75.1), turned to -90 degrees
- moved C23 3.00 mm to (196.9, 115.0), turned to 90 degrees
- moved C20 2.97 mm to (170.3, 115.2), turned to 90 degrees
- moved C24 2.67 mm to (145.7, 101.9), turned to 90 degrees
- moved C25 2.60 mm to (137.9, 105.7)
- moved C6 2.41 mm to (180.1, 79.8)
- moved C19 2.38 mm to (167.4, 114.1), turned to 90 degrees
- moved C26 2.19 mm to (137.9, 109.2)
- moved C28 2.15 mm to (143.5, 101.9), turned to 90 degrees
- moved J16 2.11 mm to (135.8, 96.0)
- moved C27 1.94 mm to (137.9, 112.7), turned to -90 degrees
- moved R1 1.93 mm to (118.4, 132.7)
- moved C29 1.90 mm to (100.2, 113.5), turned to 180 degrees
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Connections:
- J8 pad 1: /Connectors/VCC_ANT -> Net-(C31-Pad1)
Routing:
- net +3.3V: track 358.1 -> 110.5 mm, vias 2 -> 14
- net +5V: track 269.1 -> 252.0 mm
- net GND: track 100.1 -> 115.0 mm, vias 69 -> 79
- net /Connectors/PPS: track 65.0 -> 75.1 mm
- net /Connectors/1MHZ: track 74.2 -> 84.3 mm
- net /Line Drivers/SHIFT1: track 36.0 -> 45.8 mm
- net /Line Drivers/SHIFT0: track 33.0 -> 41.6 mm
- net Net-(C31-Pad1): track 0.00 -> 7.38 mm
- net /Connectors/SHIFT0_TTL: track 20.5 -> 27.7 mm
- net /Connectors/1MHZ_TTL: track 16.2 -> 22.2 mm
- net /Connectors/PPS_TTL: track 20.4 -> 26.1 mm
- net /Connectors/VCC_ANT: track 19.6 -> 15.8 mm
- net Net-(C25-Pad2): track 5.92 -> 3.02 mm
- net Net-(C25-Pad1): track 5.52 -> 2.91 mm
- net Net-(C28-Pad1): track 7.62 -> 5.09 mm
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- added copper zone on In2.Cu, net +3.3V
- added copper zone on In1.Cu, net GND
Other:
- copper layers 2 -> 4

Commit message: Increase clearance from mounting hole
Routing:
- net /Connectors/VCC_ANT: track 15.8 -> 17.9 mm
- net /Connectors/F9T_TX: track 57.9 -> 59.3 mm
Changed lines of the file:
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@@
   (segment (start 220.414 88.6) (end 215.865 88.6) (width 0.25) (layer "F.Cu") (net 20))
   (segment (start 229.57 79.29) (end 229.57 79.444) (width 0.25) (layer "F.Cu") (net 20))
+  (segment (start 216.275 73.65) (end 217.625 72.3) (width 1) (layer "F.Cu") (net 21))
   (segment (start 213.65 73.65) (end 213.625 73.625) (width 1) (layer "F.Cu") (net 21))
+  (segment (start 224.8 72.3) (end 227.57 75.07) (width 1) (layer "F.Cu") (net 21))
   (segment (start 216.275 73.65) (end 213.65 73.65) (width 1) (layer "F.Cu") (net 21))
-  (segment (start 216.275 73.65) (end 216.625 73.3) (width 1) (layer "F.Cu") (net 21))
-  (segment (start 216.625 73.3) (end 223.58 73.3) (width 1) (layer "F.Cu") (net 21))
-  (segment (start 223.58 73.3) (end 227.57 77.29) (width 1) (layer "F.Cu") (net 21))
-  (segment (start 195.104685 71.4) (end 180.886685 85.618) (width 0.25) (layer "F.Cu") (net 22))
-  (segment (start 223.68 71.4) (end 195.104685 71.4) (width 0.25) (layer "F.Cu") (net 22))
-  (segment (start 229.57 77.29) (end 223.68 71.4) (width 0.25) (layer "F.Cu") (net 22))
+  (segment (start 217.625 72.3) (end 224.8 72.3) (width 1) (layer "F.Cu") (net 21))
+  (segment (start 227.57 75.07) (end 227.57 77.29) (width 1) (layer "F.Cu") (net 21))
+  (segment (start 195.404685 71.1) (end 180.886685 85.618) (width 0.25) (layer "F.Cu") (net 22))
+  (segment (start 229.57 75.17) (end 225.5 71.1) (width 0.25) (layer "F.Cu") (net 22))
+  (segment (start 229.57 77.29) (end 229.57 75.17) (width 0.25) (layer "F.Cu") (net 22))
+  (segment (start 225.5 71.1) (end 195.404685 71.1) (width 0.25) (layer "F.Cu") (net 22))
   (segment (start 180.886685 85.618) (end 180.046 85.618) (width 0.25) (layer "F.Cu") (net 22))
   (segment (start 230.47 78.29) (end 230.545 78.215) (width 0.25) (layer "F.Cu") (net 23))
