File: d2tsf-hw.kicad_pcb (KiCad board)
At the start: 4 copper layers, 160.2 x 69.8 mm, 65 parts, among them J1 Reset MCU, J10 Serial, J11 Barrel_Jack_Switch, J12 Power, J13 RX In, J14 GND, J15 TX Out, J16 Conn_01x09_Male, J2 Programming, J3 SHIFT0, J4 SHIFT1, J5 PSS, J6 1MHZ, J7 Reset F9T, J8 ANT_VCC, J9 F9T Connector, U1 AMS1117, U2 STM32F411RETx, U3 SN74LVC8T245PWR, U4 SN74LVC8T245PWR, U5 MAX3232, Y1 16MHz

Commit message: Annotate connectors
Other:
- board text added: "1MHZ"
- board text added: "GPS Ant"
- board text added: "PSS"
- board text added: "RS232"
- board text added: "SHIFT0"
- board text added: "SHIFT1"
Changed lines of the file:
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@@
     (effects (font (size 1 1) (thickness 0.25)))
+  )
+  (gr_text "PSS" (at 190.3 136.5 90) (layer "F.SilkS")
+    (effects (font (size 1 1) (thickness 0.15)))
   )
   (gr_text "5V" (at 106.1 88.7) (layer "F.SilkS")
     (effects (font (size 3 3) (thickness 0.15)))
   )
+  (gr_text "SHIFT1" (at 176.6 135.6 90) (layer "F.SilkS")
+    (effects (font (size 1 1) (thickness 0.15)))
+  )
   (gr_text "Diamond II TimeStamp Feeder Rev0" (at 209 108.4 90) (layer "F.SilkS")
     (effects (font (size 2 2) (thickness 0.15)))
+  )
+  (gr_text "1MHZ" (at 202.6 136.2 90) (layer "F.SilkS")
+    (effects (font (size 1 1) (thickness 0.15)))
   )
   (gr_text "GND" (at 107.3 82.2) (layer "F.SilkS")
@@
     (effects (font (size 1 1) (thickness 0.15)))
   )
+  (gr_text "RS232\n" (at 129.3 119.2) (layer "F.SilkS")
+    (effects (font (size 1 1) (thickness 0.15)))
+  )
+  (gr_text "SHIFT0" (at 163.1 135.5 90) (layer "F.SilkS")
+    (effects (font (size 1 1) (thickness 0.15)))
+  )
+  (gr_text "GPS Ant" (at 236.7 137.6) (layer "F.SilkS")
+    (effects (font (size 1 1) (thickness 0.15)))
+  )

Commit message: Fix inverse numbering of programming header
Parts:
- moved J2 7.68 mm to (191.6, 91.1), turned to 180 degrees
Connections:
- J2 pad 1: GND -> +3.3V
- J2 pad 2: /Connectors/SWCLK -> /Connectors/SWDIO
- J2 pad 3: /Connectors/SWDIO -> /Connectors/SWCLK
- J2 pad 4: +3.3V -> GND
Routing:
- net GND: track 115.0 -> 111.7 mm, vias 79 -> 78
- net +3.3V: track 110.5 -> 111.2 mm
Changed lines of the file:
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@@
   )
   (footprint "Connector_PinHeader_2.54mm:PinHeader_1x04_P2.54mm_Vertical" (layer "F.Cu")
-    (at 191.5 83.46)
+    (at 191.6 91.14 180)
     (descr "Through hole straight pin header, 1x04, 2.54mm pitch, single row")
     (tags "Through hole pin header THT 1x04 2.54mm single row")
@@
     (fp_line (start 1.27 8.89) (end -1.27 8.89) (layer "F.Fab") (width 0.1))
     (fp_line (start -1.27 -0.635) (end -0.635 -1.27) (layer "F.Fab") (width 0.1))
-    (pad "1" thru_hole rect (at 0 0) (size 1.7 1.7) (drill 1) (layers *.Cu *.Mask)
-      (net 1 "GND") (pinfunction "Pin_1") (pintype "passive"))
-    (pad "2" thru_hole oval (at 0 2.54) (size 1.7 1.7) (drill 1) (layers *.Cu *.Mask)
-      (net 14 "/Connectors/SWCLK") (pinfunction "Pin_2") (pintype "passive"))
-    (pad "3" thru_hole oval (at 0 5.08) (size 1.7 1.7) (drill 1) (layers *.Cu *.Mask)
-      (net 15 "/Connectors/SWDIO") (pinfunction "Pin_3") (pintype "passive"))
-    (pad "4" thru_hole oval (at 0 7.62) (size 1.7 1.7) (drill 1) (layers *.Cu *.Mask)
-      (net 2 "+3.3V") (pinfunction "Pin_4") (pintype "passive"))
+    (pad "1" thru_hole rect (at 0 0 180) (size 1.7 1.7) (drill 1) (layers *.Cu *.Mask)
+      (net 2 "+3.3V") (pinfunction "Pin_1") (pintype "passive"))
+    (pad "2" thru_hole oval (at 0 2.54 180) (size 1.7 1.7) (drill 1) (layers *.Cu *.Mask)
+      (net 15 "/Connectors/SWDIO") (pinfunction "Pin_2") (pintype "passive"))
+    (pad "3" thru_hole oval (at 0 5.08 180) (size 1.7 1.7) (drill 1) (layers *.Cu *.Mask)
+      (net 14 "/Connectors/SWCLK") (pinfunction "Pin_3") (pintype "passive"))
+    (pad "4" thru_hole oval (at 0 7.62 180) (size 1.7 1.7) (drill 1) (layers *.Cu *.Mask)
+      (net 1 "GND") (pinfunction "Pin_4") (pintype "passive"))
     (model "${KICAD6_3DMODEL_DIR}/Connector_PinHeader_2.54mm.3dshapes/PinHeader_1x04_P2.54mm_Vertical.wrl"
       (offset (xyz 0 0 0))
@@
     (effects (font (size 1 1) (thickness 0.15)))
   )
-  (gr_text "1" (at 189.3 82.6) (layer "F.SilkS")
+  (gr_text "1" (at 193.5 92.3) (layer "F.SilkS")
     (effects (font (size 1 1) (thickness 0.15)))
   )
@@
   )
   (segment (start 156 93) (end 156 89.475) (width 0.25) (layer "F.Cu") (net 1))
-  (segment (start 194.797 83.46) (end 194.818 83.439) (width 0.25) (layer "F.Cu") (net 1))
   (segment (start 165.876777 85.423223) (end 163.878858 85.423223) (width 0.25) (layer "F.Cu") (net 1))
   (segment (start 181.482 83.618) (end 180.046 83.618) (width 0.25) (layer "F.Cu") (net 1))
@@
   (segment (start 165.7 115.2) (end 165.735 115.235) (width 0.25) (layer "F.Cu") (net 1))
   (segment (start 160.475 123.825) (end 159.5 124.8) (width 0.25) (layer "F.Cu") (net 1))
-  (segment (start 191.5 83.46) (end 194.797 83.46) (width 0.25) (layer "F.Cu") (net 1))
   (segment (start 115.1 99.8) (end 115.1 97.1) (width 0.25) (layer "F.Cu") (net 1))
   (segment (start 111.125 97.028) (end 111.125 99.744) (width 0.25) (layer "F.Cu") (net 1))
@@
   (via (at 170.3 111.7) (size 0.8) (drill 0.4) (layers "F.Cu" "B.Cu") (net 1))
   (via (at 168.8 76.4) (size 0.8) (drill 0.4) (layers "F.Cu" "B.Cu") (net 1))
-  (via (at 194.818 83.439) (size 0.8) (drill 0.4) (layers "F.Cu" "B.Cu") (net 1))
   (via (at 178.8 118.7) (size 0.8) (drill 0.4) (layers "F.Cu" "B.Cu") (free) (net 1))
   (via (at 178.181 94.615) (size 0.8) (drill 0.4) (layers "F.Cu" "B.Cu") (net 1))
@@
   (segment (start 133.23 75.63) (end 135.8 75.63) (width 0.25) (layer "B.Cu") (net 1))
   (segment (start 183.45 92.65) (end 183.5 92.7) (width 0.3) (layer "F.Cu") (net 2))
-  (segment (start 189.02 91.08) (end 189 91.1) (width 0.3) (layer "F.Cu") (net 2))
   (segment (start 188.1 116.395) (end 188.13 116.425) (width 0.3) (layer "F.Cu") (net 2))
   (segment (start 110.846 102.973) (end 111.125 102.694) (width 0.3) (layer "F.Cu") (net 2))
@@
   (segment (start 165.968 83.118) (end 165.6 82.75) (width 0.25) (layer "F.Cu") (net 2))
   (segment (start 170.6 78.35) (end 169.35 78.35) (width 0.3) (layer "F.Cu") (net 2))
+  (segment (start 191.6 91.14) (end 188.44 91.14) (width 0.3) (layer "F.Cu") (net 2))
+  (segment (start 188.44 91.14) (end 188.4 91.1) (width 0.3) (layer "F.Cu") (net 2))
   (segment (start 186.1125 116.6875) (end 186.375 116.425) (width 0.3) (layer "F.Cu") (net 2))
   (segment (start 158.8 116.8875) (end 159.7125 116.8875) (width 0.3) (layer "F.Cu") (net 2))
-  (segment (start 191.5 91.08) (end 189.02 91.08) (width 0.3) (layer "F.Cu") (net 2))
   (segment (start 168.8 96.459) (end 171.591 96.459) (width 0.3) (layer "F.Cu") (net 2))
   (segment (start 110.846 107.696) (end 113.596 107.696) (width 0.3) (layer "F.Cu") (net 2))
@@
   (segment (start 164.35 82.75) (end 163.7 82.1) (width 0.3) (layer "F.Cu") (net 2))
   (segment (start 162.8 96.45) (end 166.107 96.45) (width 0.3) (layer "F.Cu") (net 2))
-  (via (at 189 91.1) (size 0.8) (drill 0.4) (layers "F.Cu" "B.Cu") (net 2))
+  (via (at 188.4 91.1) (size 0.8) (drill 0.4) (layers "F.Cu" "B.Cu") (net 2))
   (via (at 125 129.7) (size 0.8) (drill 0.4) (layers "F.Cu" "B.Cu") (net 2))
   (via (at 156 84.6) (size 0.8) (drill 0.4) (layers "F.Cu" "B.Cu") (net 2))
@@
   (segment (start 119.3275 132.715) (end 119.3125 132.7) (width 0.25) (layer "F.Cu") (net 13))
   (segment (start 122.5 132.715) (end 119.3275 132.715) (width 0.25) (layer "F.Cu") (net 13))
-  (segment (start 185.018 86) (end 191.5 86) (width 0.25) (layer "F.Cu") (net 14))
-  (segment (start 180.046 89.618) (end 181.4 89.618) (width 0.25) (layer "F.Cu") (net 14))
-  (segment (start 181.4 89.618) (end 185.018 86) (width 0.25) (layer "F.Cu") (net 14))
-  (segment (start 183.24 88.54) (end 191.5 88.54) (width 0.25) (layer "F.Cu") (net 15))
-  (segment (start 181.662 90.118) (end 183.24 88.54) (width 0.25) (layer "F.Cu") (net 15))
-  (segment (start 180.046 90.118) (end 181.662 90.118) (width 0.25) (layer "F.Cu") (net 15))
+  (segment (start 184.958 86.06) (end 181.4 89.618) (width 0.25) (layer "F.Cu") (net 14))
+  (segment (start 181.4 89.618) (end 180.046 89.618) (width 0.25) (layer "F.Cu") (net 14))
+  (segment (start 191.6 86.06) (end 184.958 86.06) (width 0.25) (layer "F.Cu") (net 14))
+  (segment (start 181.722 90.118) (end 183.24 88.6) (width 0.25) (layer "F.Cu") (net 15))
+  (segment (start 180.046 90.118) (end 181.722 90.118) (width 0.25) (layer "F.Cu") (net 15))
+  (segment (start 191.6 88.6) (end 183.3 88.6) (width 0.25) (layer "F.Cu") (net 15))
   (segment (start 169.025 119.925) (end 169.1 120) (width 0.25) (layer "F.Cu") (net 16))
   (segment (start 167.37 120.575) (end 168.625 120.575) (width 0.25) (layer "F.Cu") (net 16))

Commit message: Fix wrong connection of SWD pins
Parts:
- moved J2 17.5 mm to (187.7, 74.1), turned to -90 degrees
Connections:
- U2 pad 34: /Connectors/SWDIO -> unconnected-(U2-Pad34)
- U2 pad 35: /Connectors/SWCLK -> unconnected-(U2-Pad35)
- U2 pad 46: unconnected-(U2-Pad46) -> /Connectors/SWDIO
- U2 pad 49: unconnected-(U2-Pad49) -> /Connectors/SWCLK
Routing:
- net /Connectors/SWCLK: track 13.0 -> 9.22 mm
- net GND: track 111.7 -> 110.5 mm
- net +3.3V: track 111.2 -> 110.5 mm
- net /Connectors/SWDIO: track 12.1 -> 12.8 mm

Commit message: Release board rev1
Ferrite bead 1 was removed (not needed)
Parts:
- removed FB1: 33uH, Capacitor_SMD:C_0805_2012Metric
Connections:
- C31 pad 1: Net-(C31-Pad1) -> /Connectors/VCC_ANT
- J8 pad 1: Net-(C31-Pad1) -> /Connectors/VCC_ANT
Routing:
- net /Connectors/VCC_ANT: track 17.9 -> 27.1 mm
- net Net-(C31-Pad1): track 7.38 -> 0.00 mm
Other:
- board text added: "Diamond II TimeStamp Feeder Rev1"
- board text removed: "Diamond II TimeStamp Feeder Rev0"

Commit message: Add pull up resistors to SWD signals
Parts:
- added R4: 10k, Resistor_SMD:R_0805_2012Metric, F.Cu at (182.9, 77.8)
- added R5: 10k, Resistor_SMD:R_0805_2012Metric, F.Cu at (175.5, 76.3)
- J2: value Programming -> Prog
Routing:
- net +3.3V: track 110.5 -> 113.6 mm, vias 14 -> 16
- net /Connectors/SWCLK: track 9.22 -> 12.3 mm
- net /Connectors/SWDIO: track 12.8 -> 15.1 mm
Changed lines of the file:
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@@
     )
   )
+  (footprint "Resistor_SMD:R_0805_2012Metric" (layer "F.Cu")
+    (at 175.5 76.3)
+    (descr "Resistor SMD 0805 (2012 Metric), square (rectangular) end terminal, IPC_7351 nominal, (Body size source: IPC-SM-782 page 72, https://www.pcb-3d.com/wordpress/wp-content/uploads/ipc-sm-782a_amendment_1_and_2.pdf), generated with kicad-footprint-generator")
+    (tags "resistor")
+    (property "Sheetfile" "connectors.kicad_sch")
+    (property "Sheetname" "Connectors")
+    (attr smd)
+    (fp_text reference "R5" (at 0 -1.65) (layer "F.SilkS")
+      (effects (font (size 1 1) (thickness 0.15)))
+    )
+    (fp_text value "10k" (at 0 1.65) (layer "F.Fab")
+      (effects (font (size 1 1) (thickness 0.15)))
+    )
+    (fp_text user "${REFERENCE}" (at 0 0) (layer "F.Fab")
+      (effects (font (size 0.5 0.5) (thickness 0.08)))
+    )
+    (fp_line (start -0.227064 -0.735) (end 0.227064 -0.735) (layer "F.SilkS") (width 0.12))
+    (fp_line (start -0.227064 0.735) (end 0.227064 0.735) (layer "F.SilkS") (width 0.12))
+    (fp_line (start 1.68 0.95) (end -1.68 0.95) (layer "F.CrtYd") (width 0.05))
+    (fp_line (start -1.68 0.95) (end -1.68 -0.95) (layer "F.CrtYd") (width 0.05))
+    (fp_line (start -1.68 -0.95) (end 1.68 -0.95) (layer "F.CrtYd") (width 0.05))
+    (fp_line (start 1.68 -0.95) (end 1.68 0.95) (layer "F.CrtYd") (width 0.05))
+    (fp_line (start 1 0.625) (end -1 0.625) (layer "F.Fab") (width 0.1))
+    (fp_line (start -1 0.625) (end -1 -0.625) (layer "F.Fab") (width 0.1))
+    (fp_line (start 1 -0.625) (end 1 0.625) (layer "F.Fab") (width 0.1))
+    (fp_line (start -1 -0.625) (end 1 -0.625) (layer "F.Fab") (width 0.1))
+    (pad "1" smd roundrect (at -0.9125 0) (size 1.025 1.4) (layers "F.Cu" "F.Paste" "F.Mask") (roundrect_rratio 0.243902)
+      (net 2 "+3.3V") (pintype "passive"))
+    (pad "2" smd roundrect (at 0.9125 0) (size 1.025 1.4) (layers "F.Cu" "F.Paste" "F.Mask") (roundrect_rratio 0.243902)
+      (net 14 "/Connectors/SWCLK") (pintype "passive"))
+    (model "${KICAD6_3DMODEL_DIR}/Resistor_SMD.3dshapes/R_0805_2012Metric.wrl"
+      (offset (xyz 0 0 0))
+      (scale (xyz 1 1 1))
+      (rotate (xyz 0 0 0))
+    )
+  )
   (footprint "Capacitor_SMD:C_0805_2012Metric" (layer "F.Cu")
     (at 170.6 77.4 90)
@@
     )
   )
+  (footprint "Resistor_SMD:R_0805_2012Metric" (layer "F.Cu")
+    (at 182.9 77.8 90)
+    (descr "Resistor SMD 0805 (2012 Metric), square (rectangular) end terminal, IPC_7351 nominal, (Body size source: IPC-SM-782 page 72, https://www.pcb-3d.com/wordpress/wp-content/uploads/ipc-sm-782a_amendment_1_and_2.pdf), generated with kicad-footprint-generator")
+    (tags "resistor")
+    (property "Sheetfile" "connectors.kicad_sch")
+    (property "Sheetname" "Connectors")
+    (attr smd)
+    (fp_text reference "R4" (at -2.6 0.7 90) (layer "F.SilkS")
+      (effects (font (size 1 1) (thickness 0.15)))
+    )
+    (fp_text value "10k" (at 0 1.65 90) (layer "F.Fab")
+      (effects (font (size 1 1) (thickness 0.15)))
+    )
+    (fp_text user "${REFERENCE}" (at 0 0 90) (layer "F.Fab")
+      (effects (font (size 0.5 0.5) (thickness 0.08)))
+    )
+    (fp_line (start -0.227064 0.735) (end 0.227064 0.735) (layer "F.SilkS") (width 0.12))
+    (fp_line (start -0.227064 -0.735) (end 0.227064 -0.735) (layer "F.SilkS") (width 0.12))
+    (fp_line (start -1.68 -0.95) (end 1.68 -0.95) (layer "F.CrtYd") (width 0.05))
+    (fp_line (start 1.68 0.95) (end -1.68 0.95) (layer "F.CrtYd") (width 0.05))
+    (fp_line (start -1.68 0.95) (end -1.68 -0.95) (layer "F.CrtYd") (width 0.05))
+    (fp_line (start 1.68 -0.95) (end 1.68 0.95) (layer "F.CrtYd") (width 0.05))
+    (fp_line (start -1 -0.625) (end 1 -0.625) (layer "F.Fab") (width 0.1))
+    (fp_line (start 1 -0.625) (end 1 0.625) (layer "F.Fab") (width 0.1))
+    (fp_line (start 1 0.625) (end -1 0.625) (layer "F.Fab") (width 0.1))
+    (fp_line (start -1 0.625) (end -1 -0.625) (layer "F.Fab") (width 0.1))
+    (pad "1" smd roundrect (at -0.9125 0 90) (size 1.025 1.4) (layers "F.Cu" "F.Paste" "F.Mask") (roundrect_rratio 0.243902)
+      (net 2 "+3.3V") (pintype "passive"))
+    (pad "2" smd roundrect (at 0.9125 0 90) (size 1.025 1.4) (layers "F.Cu" "F.Paste" "F.Mask") (roundrect_rratio 0.243902)
+      (net 15 "/Connectors/SWDIO") (pintype "passive"))
+    (model "${KICAD6_3DMODEL_DIR}/Resistor_SMD.3dshapes/R_0805_2012Metric.wrl"
+      (offset (xyz 0 0 0))
+      (scale (xyz 1 1 1))
+      (rotate (xyz 0 0 0))
+    )
+  )
   (footprint "Capacitor_SMD:C_0805_2012Metric" (layer "F.Cu")
     (at 168.8 97.409 -90)
@@
     (property "Sheetname" "MCU")
     (attr smd)
-    (fp_text reference "C6" (at 2.7 1.1 90) (layer "F.SilkS")
+    (fp_text reference "C6" (at -2.2 1.6 90) (layer "F.SilkS")
       (effects (font (size 1 1) (thickness 0.15)))
     )
-    (fp_text value "100n" (at 0 1.68 90) (layer "F.Fab")
+    (fp_text value "100n" (at 1.6 -1.7 270) (layer "F.Fab")
       (effects (font (size 1 1) (thickness 0.15)))
     )
@@
       (effects (font (size 1 1) (thickness 0.15)))
     )
-    (fp_text value "Programming" (at 3.4 0.5) (layer "F.SilkS")
+    (fp_text value "Prog" (at -2.5 0.5) (layer "F.SilkS")
       (effects (font (size 1 1) (thickness 0.15)))
     )
@@
   (segment (start 178.228 92.65) (end 178.121 92.543) (width 0.3) (layer "F.Cu") (net 2))
   (segment (start 171.794 94.441695) (end 171.794 96.369) (width 0.25) (layer "F.Cu") (net 2))
+  (segment (start 182.9 78.7125) (end 184.3875 78.7125) (width 0.3) (layer "F.Cu") (net 2))
   (segment (start 159.925 116.675) (end 161.63 116.675) (width 0.3) (layer "F.Cu") (net 2))
   (segment (start 185.1 114.9) (end 185.15 114.85) (width 0.3) (layer "F.Cu") (net 2))
@@
   (segment (start 125.04 132.715) (end 125.04 129.74) (width 0.3) (layer "F.Cu") (net 2))
   (segment (start 168.8 96.459) (end 168.8 95.5) (width 0.3) (layer "F.Cu") (net 2))
+  (segment (start 184.3875 78.7125) (end 184.4 78.7) (width 0.3) (layer "F.Cu") (net 2))
   (segment (start 158.8 116.8875) (end 158.8 115.2) (width 0.3) (layer "F.Cu") (net 2))
   (segment (start 159.7125 116.8875) (end 159.925 116.675) (width 0.3) (layer "F.Cu") (net 2))
@@
   (segment (start 110.846 107.696) (end 110.846 102.973) (width 0.3) (layer "F.Cu") (net 2))
   (segment (start 182.35 80.75) (end 182.4 80.7) (width 0.3) (layer "F.Cu") (net 2))
+  (segment (start 174.5875 76.3) (end 172.9 76.3) (width 0.3) (layer "F.Cu") (net 2))
   (segment (start 145.7 102.85) (end 148.45 102.85) (width 0.3) (layer "F.Cu") (net 2))
   (segment (start 170.621 81.193) (end 170.621 78.371) (width 0.3) (layer "F.Cu") (net 2))
@@
   (segment (start 164.35 82.75) (end 163.7 82.1) (width 0.3) (layer "F.Cu") (net 2))
   (segment (start 162.8 96.45) (end 166.107 96.45) (width 0.3) (layer "F.Cu") (net 2))
+  (via (at 172.9 76.3) (size 0.8) (drill 0.4) (layers "F.Cu" "B.Cu") (net 2))
   (via (at 187.7 76.6) (size 0.8) (drill 0.4) (layers "F.Cu" "B.Cu") (net 2))
   (via (at 125 129.7) (size 0.8) (drill 0.4) (layers "F.Cu" "B.Cu") (net 2))
@@
   (via (at 169.4 94.9) (size 0.8) (drill 0.4) (layers "F.Cu" "B.Cu") (net 2))
   (via (at 158.9 115.1) (size 0.8) (drill 0.4) (layers "F.Cu" "B.Cu") (net 2))
+  (via (at 184.4 78.7) (size 0.8) (drill 0.4) (layers "F.Cu" "B.Cu") (net 2))
   (via (at 162.8 94.6) (size 0.8) (drill 0.4) (layers "F.Cu" "B.Cu") (net 2))
   (via (at 182.4 80.7) (size 0.8) (drill 0.4) (layers "F.Cu" "B.Cu") (net 2))
@@
   (segment (start 122.5 132.715) (end 119.3275 132.715) (width 0.25) (layer "F.Cu") (net 13))
   (segment (start 182.174695 74.1) (end 182.62 74.1) (width 0.25) (layer "F.Cu") (net 14))
+  (segment (start 176.4125 76.3) (end 178.5 76.3) (width 0.25) (layer "F.Cu") (net 14))
+  (segment (start 178.5 76.3) (end 179.237347 77.037347) (width 0.25) (layer "F.Cu") (net 14))
   (segment (start 178.121 81.193) (end 178.121 78.153695) (width 0.25) (layer "F.Cu") (net 14))
-  (segment (start 178.121 78.153695) (end 182.174695 74.1) (width 0.25) (layer "F.Cu") (net 14))
+  (segment (start 179.237347 77.037347) (end 182.174695 74.1) (width 0.25) (layer "F.Cu") (net 14))
+  (segment (start 178.121 78.153695) (end 179.237347 77.037347) (width 0.25) (layer "F.Cu") (net 14))
   (segment (start 181.182 84.118) (end 185.16 80.14) (width 0.25) (layer "F.Cu") (net 15))
   (segment (start 180.046 84.118) (end 181.182 84.118) (width 0.25) (layer "F.Cu") (net 15))
-  (segment (start 185.16 80.14) (end 185.16 74.1) (width 0.25) (layer "F.Cu") (net 15))
+  (segment (start 185.16 80.14) (end 185.16 76.76) (width 0.25) (layer "F.Cu") (net 15))
+  (segment (start 185.16 76.76) (end 185.16 74.1) (width 0.25) (layer "F.Cu") (net 15))
+  (segment (start 185.0325 76.8875) (end 185.16 76.76) (width 0.25) (layer "F.Cu") (net 15))
+  (segment (start 182.9 76.8875) (end 185.0325 76.8875) (width 0.25) (layer "F.Cu") (net 15))
   (segment (start 169.025 119.925) (end 169.1 120) (width 0.25) (layer "F.Cu") (net 16))
   (segment (start 167.37 120.575) (end 168.625 120.575) (width 0.25) (layer "F.Cu") (net 16))

Commit message: Mark microcontroller pin 1 on silkscreen
Routing:
- net GND: vias 78 -> 80
Changed lines of the file:
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@@
     (effects (font (size 3 3) (thickness 0.15)))
+  )
+  (gr_text "1" (at 167.1 82.4) (layer "F.SilkS")
+    (effects (font (size 1 1) (thickness 0.15)))
   )
   (gr_text "SHIFT1" (at 176.6 135.6 90) (layer "F.SilkS")
@@
   (via (at 171.7 85.1) (size 0.8) (drill 0.4) (layers "F.Cu" "B.Cu") (free) (net 1))
   (via (at 100 123.9) (size 0.8) (drill 0.4) (layers "F.Cu" "B.Cu") (free) (net 1))
+  (via (at 226.6 87.4) (size 0.8) (drill 0.4) (layers "F.Cu" "B.Cu") (free) (net 1))
   (via (at 177.3 74.1) (size 0.8) (drill 0.4) (layers "F.Cu" "B.Cu") (net 1))
   (via (at 193.9 111.4) (size 0.8) (drill 0.4) (layers "F.Cu" "B.Cu") (net 1))
@@
   (via (at 207.6 82) (size 0.8) (drill 0.4) (layers "F.Cu" "B.Cu") (free) (net 1))
   (via (at 212.275 76.625) (size 0.8) (drill 0.4) (layers "F.Cu" "B.Cu") (net 1))
+  (via (at 230.1 83.9) (size 0.8) (drill 0.4) (layers "F.Cu" "B.Cu") (free) (net 1))
   (via (at 129.8 91.8) (size 0.8) (drill 0.4) (layers "F.Cu" "B.Cu") (free) (net 1))
   (via (at 192.1 115.1) (size 0.8) (drill 0.4) (layers "F.Cu" "B.Cu") (net 1))
