File: d2tsf-hw.kicad_pcb (KiCad board)
At the start: 4 copper layers, 160.2 x 69.8 mm, 66 parts, among them J1 Reset MCU, J10 Serial, J11 Barrel_Jack_Switch, J12 Power, J13 RX In, J14 GND, J15 TX Out, J16 Conn_01x09_Male, J2 Prog, J3 SHIFT0, J4 SHIFT1, J5 PSS, J6 1MHZ, J7 Reset F9T, J8 ANT_VCC, J9 F9T Connector, U1 AMS1117, U2 STM32F411RETx, U3 SN74LVC8T245PWR, U4 SN74LVC8T245PWR, U5 MAX3232, Y1 16MHz

Commit message: Rev3: Fix GPS receiver start problem and update to KiCad 7
- Pin TP2 of GPS receiver seems to be pulled down briefly at start time,
  this triggers the safe boot mode. A buffer was added to address this
  issue. Thanks Chris C. for the fix and thanks Paul H. for the
  investigation
- All files were adapted to KiCad 7 format and many symbols and footprints
  were replaced with newer ones.
Parts:
- added U6: 74LVC1G125, Package_TO_SOT_SMD:SOT-23-5_HandSoldering, F.Cu at (228.6, 86.9)
- added U7: 74LVC1G125, Package_TO_SOT_SMD:SOT-23-5_HandSoldering, F.Cu at (234.4, 86.9)
- J2: value Prog -> Programming
- U3, U4: footprint footprints:SOP65P640X120-24N -> Package_SO:TSSOP-24_4.4x7.8mm_P0.65mm
- U5: footprint footprints:SOIC127P600X175-16N -> Package_SO:SOIC-16_3.9x9.9mm_P1.27mm
- moved R5 6.77 mm to (181.9, 78.6), turned to 90 degrees
- moved R4 1.29 mm to (183.9, 78.6)
- moved C6 0.27 mm to (179.8, 79.8)
Connections:
- TP3 pad 1: /Connectors/PPS -> Net-(U4-A1)
- TP4 pad 1: /Connectors/1MHZ -> Net-(U4-A5)
- U4 pad 10: /Connectors/1MHZ -> Net-(U4-A5)
- U4 pad 3: /Connectors/PPS -> Net-(U4-A1)
- U4 pad 4: /Connectors/PPS -> Net-(U4-A1)
- U4 pad 5: /Connectors/PPS -> Net-(U4-A1)
- U4 pad 6: /Connectors/PPS -> Net-(U4-A1)
- U4 pad 7: /Connectors/1MHZ -> Net-(U4-A5)
- U4 pad 8: /Connectors/1MHZ -> Net-(U4-A5)
- U4 pad 9: /Connectors/1MHZ -> Net-(U4-A5)
Routing:
- net Net-(U4-A5): track 0.00 -> 75.4 mm
- net /Connectors/1MHZ: track 84.3 -> 10.3 mm
- net Net-(U4-A1): track 0.00 -> 67.7 mm
- net /Connectors/PPS: track 75.1 -> 7.46 mm
- net GND: track 110.5 -> 60.0 mm, vias 80 -> 66
- net +3.3V: track 113.6 -> 117.2 mm
- net B4: track 44.6 -> 41.8 mm
- net B5: track 43.0 -> 40.9 mm
- net B3: track 45.3 -> 44.0 mm
- net /Connectors/SWDIO: track 15.1 -> 14.3 mm
- net /Connectors/SWCLK: track 12.3 -> 11.6 mm
- net /Connectors/1MHZ_TTL: track 22.2 -> 22.9 mm
- net B2: track 46.1 -> 45.6 mm
- net Net-(J13-Pin_3): track 38.2 -> 38.8 mm
Other:
- board text added: "Diamond II TimeStamp Feeder Rev2"
- board text removed: "Diamond II TimeStamp Feeder Rev1"

Commit message: Add metadata to follow Diamond's standard and use a letter for the revision
Other:
- board text added: "Diamond II TimeStamp Feeder RevB"
- board text removed: "Diamond II TimeStamp Feeder Rev2"
Changed lines of the file:
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@@
     (effects (font (size 1 1) (thickness 0.15)))
   )
-  (gr_text "Diamond II TimeStamp Feeder Rev2" (at 209 108.4 90) (layer "F.SilkS")
+  (gr_text "Diamond II TimeStamp Feeder RevB" (at 209 108.4 90) (layer "F.SilkS")
     (effects (font (size 2 2) (thickness 0.15)))
   )
