File: line_drivers.kicad_sch (KiCad schematic)
At the start: 16 parts, among them U3 SN74LVC8T245PWR, U4 SN74LVC8T245PWR, U5 MAX3232

Commit message: Change to use 4 layers
- In1 is GND layer
- In2 is 3.3V layer
- Additionally, a few test points were added
Parts:
- added TP1: SHIFT0, TestPoint:TestPoint_Pad_D1.0mm, symbol Connector:TestPoint
- added TP2: SHIFT1, TestPoint:TestPoint_Pad_D1.0mm, symbol Connector:TestPoint
- added TP3: PPS, TestPoint:TestPoint_Pad_D1.0mm, symbol Connector:TestPoint
- added TP4: 1MHZ, TestPoint:TestPoint_Pad_D1.0mm, symbol Connector:TestPoint
Connections:
- net 1MHZ: now also TP4.1
- net PPS: now also TP3.1
- net SHIFT0: now also TP1.1
- net SHIFT1: now also TP2.1
Changed lines of the file:
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@@
   (junction (at 232.41 35.56) (diameter 0) (color 0 0 0 0)
   )
+  (junction (at 160.02 64.77) (diameter 0) (color 0 0 0 0)
+  )
   (junction (at 93.98 27.94) (diameter 0) (color 0 0 0 0)
   )
@@
   (junction (at 232.41 27.94) (diameter 0) (color 0 0 0 0)
   )
+  (junction (at 43.18 74.93) (diameter 0) (color 0 0 0 0)
+  )
   (junction (at 86.36 67.31) (diameter 0) (color 0 0 0 0)
   )
@@
   )
   (junction (at 115.57 35.56) (diameter 0) (color 0 0 0 0)
+  )
+  (junction (at 43.18 64.77) (diameter 0) (color 0 0 0 0)
+  )
+  (junction (at 160.02 74.93) (diameter 0) (color 0 0 0 0)
   )
   (junction (at 86.36 77.47) (diameter 0) (color 0 0 0 0)
@@
     (stroke (width 0) (type default) (color 0 0 0 0))
   )
+  (wire (pts (xy 160.02 74.93) (xy 163.83 74.93))
+    (stroke (width 0) (type default) (color 0 0 0 0))
+  )
   (wire (pts (xy 43.18 154.94) (xy 49.53 154.94))
     (stroke (width 0) (type default) (color 0 0 0 0))
@@
     (stroke (width 0) (type default) (color 0 0 0 0))
   )
+  (wire (pts (xy 43.18 64.77) (xy 48.26 64.77))
+    (stroke (width 0) (type default) (color 0 0 0 0))
+  )
   (wire (pts (xy 201.93 72.39) (xy 204.47 72.39))
     (stroke (width 0) (type default) (color 0 0 0 0))
@@
     (stroke (width 0) (type default) (color 0 0 0 0))
   )
-  (wire (pts (xy 156.21 74.93) (xy 163.83 74.93))
+  (wire (pts (xy 156.21 74.93) (xy 160.02 74.93))
     (stroke (width 0) (type default) (color 0 0 0 0))
   )
@@
     (stroke (width 0) (type default) (color 0 0 0 0))
   )
-  (wire (pts (xy 40.64 74.93) (xy 48.26 74.93))
+  (wire (pts (xy 40.64 74.93) (xy 43.18 74.93))
     (stroke (width 0) (type default) (color 0 0 0 0))
   )
@@
     (stroke (width 0) (type default) (color 0 0 0 0))
   )
+  (wire (pts (xy 160.02 64.77) (xy 163.83 64.77))
+    (stroke (width 0) (type default) (color 0 0 0 0))
+  )
   (wire (pts (xy 232.41 27.94) (xy 237.49 27.94))
     (stroke (width 0) (type default) (color 0 0 0 0))
@@
     (stroke (width 0) (type default) (color 0 0 0 0))
   )
-  (wire (pts (xy 40.64 64.77) (xy 48.26 64.77))
+  (wire (pts (xy 40.64 64.77) (xy 43.18 64.77))
     (stroke (width 0) (type default) (color 0 0 0 0))
   )
@@
     (stroke (width 0) (type default) (color 0 0 0 0))
   )
+  (wire (pts (xy 43.18 74.93) (xy 48.26 74.93))
+    (stroke (width 0) (type default) (color 0 0 0 0))
+  )
   (wire (pts (xy 163.83 72.39) (xy 163.83 69.85))
     (stroke (width 0) (type default) (color 0 0 0 0))
@@
     (stroke (width 0) (type default) (color 0 0 0 0))
   )
-  (wire (pts (xy 156.21 64.77) (xy 163.83 64.77))
+  (wire (pts (xy 156.21 64.77) (xy 160.02 64.77))
     (stroke (width 0) (type default) (color 0 0 0 0))
   )
@@
     (pin "2")
   )
+  (symbol (lib_id "Connector:TestPoint") (at 160.02 74.93 180) (unit 1)
+    (in_bom yes) (on_board yes)
+    (property "Reference" "TP4" (id 0) (at 154.94 78.74 0)
+      (effects (font (size 1.27 1.27)) (justify right))
+    )
+    (property "Value" "1MHZ" (id 1) (at 153.67 81.28 0)
+      (effects (font (size 1.27 1.27)) (justify right))
+    )
+    (property "Footprint" "TestPoint:TestPoint_Pad_D1.0mm" (id 2) (at 154.94 74.93 0)
+      (effects (font (size 1.27 1.27)) hide)
+    )
+    (property "Datasheet" "~" (id 3) (at 154.94 74.93 0)
+      (effects (font (size 1.27 1.27)) hide)
+    )
+    (pin "1")
+  )
   (symbol (lib_id "power:GND") (at 110.49 125.73 0) (unit 1)
     (in_bom yes) (on_board yes) (fields_autoplaced)
@@
     )
     (property "Datasheet" "" (id 3) (at 210.82 35.56 0)
+      (effects (font (size 1.27 1.27)) hide)
+    )
+    (pin "1")
+  )
+  (symbol (lib_id "Connector:TestPoint") (at 43.18 74.93 180) (unit 1)
+    (in_bom yes) (on_board yes)
+    (property "Reference" "TP2" (id 0) (at 38.1 77.47 0)
+      (effects (font (size 1.27 1.27)) (justify right))
+    )
+    (property "Value" "SHIFT1" (id 1) (at 36.83 80.01 0)
+      (effects (font (size 1.27 1.27)) (justify right))
+    )
+    (property "Footprint" "TestPoint:TestPoint_Pad_D1.0mm" (id 2) (at 38.1 74.93 0)
+      (effects (font (size 1.27 1.27)) hide)
+    )
+    (property "Datasheet" "~" (id 3) (at 38.1 74.93 0)
       (effects (font (size 1.27 1.27)) hide)
     )
@@
       (effects (font (size 1.27 1.27)) hide)
     )
+    (pin "1")
+  )
+  (symbol (lib_id "Connector:TestPoint") (at 43.18 64.77 180) (unit 1)
+    (in_bom yes) (on_board yes)
+    (property "Reference" "TP1" (id 0) (at 38.1 68.58 0)
+      (effects (font (size 1.27 1.27)) (justify right))
+    )
+    (property "Value" "SHIFT0" (id 1) (at 38.1 71.12 0)
+      (effects (font (size 1.27 1.27)) (justify right))
+    )
+    (property "Footprint" "TestPoint:TestPoint_Pad_D1.0mm" (id 2) (at 38.1 64.77 0)
+      (effects (font (size 1.27 1.27)) hide)
+    )
+    (property "Datasheet" "~" (id 3) (at 38.1 64.77 0)
+      (effects (font (size 1.27 1.27)) hide)
+    )
+    (pin "1")
+  )
+  (symbol (lib_id "Connector:TestPoint") (at 160.02 64.77 180) (unit 1)
+    (in_bom yes) (on_board yes)
+    (property "Reference" "TP3" (id 0) (at 154.94 67.31 0)
+      (effects (font (size 1.27 1.27)) (justify right))
+    )
+    (property "Value" "PPS" (id 1) (at 154.94 69.85 0)
+      (effects (font (size 1.27 1.27)) (justify right))
+    )
+    (property "Footprint" "TestPoint:TestPoint_Pad_D1.0mm" (id 2) (at 154.94 64.77 0)
+      (effects (font (size 1.27 1.27)) hide)
+    )
+    (property "Datasheet" "~" (id 3) (at 154.94 64.77 0)
+      (effects (font (size 1.27 1.27)) hide)
+    )
