File: mcu.kicad_sch (KiCad schematic)
At the start: 16 parts, among them J1 Reset MCU, U2 STM32F411RETx, Y1 16MHz

Commit message: Change to use 4 layers
- In1 is GND layer
- In2 is 3.3V layer
- Additionally, a few test points were added
Parts:
- C11: value 10p -> 10n
Changed lines of the file:
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@@
       (effects (font (size 1.27 1.27)) (justify left))
     )
-    (property "Value" "10p" (id 1) (at 179.07 58.4199 0)
+    (property "Value" "10n" (id 1) (at 179.07 58.4199 0)
       (effects (font (size 1.27 1.27)) (justify left))
     )

Commit message: Fix wrong connection of SWD pins
Connections:
- net SWCLK: now also U2.49 (PA14); no longer U2.35 (PB14)
- net SWDIO: now also U2.46 (PA13); no longer U2.34 (PB13)
Changed lines of the file:
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@@
   (junction (at 68.58 45.72) (diameter 0) (color 0 0 0 0)
   )
+  (no_connect (at 161.29 149.86))
   (no_connect (at 161.29 93.98))
-  (no_connect (at 161.29 109.22))
   (no_connect (at 125.73 124.46))
   (no_connect (at 125.73 139.7))
-  (no_connect (at 161.29 106.68))
   (no_connect (at 125.73 129.54))
   (no_connect (at 161.29 91.44))
@@
   (no_connect (at 125.73 137.16))
   (no_connect (at 161.29 76.2))
+  (no_connect (at 161.29 147.32))
   (no_connect (at 125.73 121.92))
   (no_connect (at 161.29 137.16))
@@
     (stroke (width 0) (type default) (color 0 0 0 0))
   )
+  (wire (pts (xy 161.29 109.22) (xy 166.37 109.22))
+    (stroke (width 0) (type default) (color 0 0 0 0))
+  )
   (wire (pts (xy 160.02 50.8) (xy 173.99 50.8))
     (stroke (width 0) (type default) (color 0 0 0 0))
@@
   )
   (wire (pts (xy 140.97 33.02) (xy 140.97 68.58))
+    (stroke (width 0) (type default) (color 0 0 0 0))
+  )
+  (wire (pts (xy 161.29 106.68) (xy 166.37 106.68))
     (stroke (width 0) (type default) (color 0 0 0 0))
   )
@@
     )
   )
-  (hierarchical_label "SWDIO" (shape input) (at 161.29 147.32 0)
+  (hierarchical_label "SWDIO" (shape input) (at 166.37 106.68 0)
     (effects (font (size 1.27 1.27)) (justify left))
   )
@@
     (effects (font (size 1.27 1.27)) (justify left))
   )
-  (hierarchical_label "SWCLK" (shape input) (at 161.29 149.86 0)
-    (effects (font (size 1.27 1.27)) (justify left))
-  )
+  (hierarchical_label "SWCLK" (shape input) (at 166.37 109.22 0)
+    (effects (font (size 1.27 1.27)) (justify left))
+  )
