File: mcu.kicad_sch (KiCad schematic)
At the start: 16 parts, among them J1 Reset MCU, U2 STM32F411RETx, Y1 16MHz

Commit message: Rev3: Fix GPS receiver start problem and update to KiCad 7
- Pin TP2 of GPS receiver seems to be pulled down briefly at start time,
  this triggers the safe boot mode. A buffer was added to address this
  issue. Thanks Chris C. for the fix and thanks Paul H. for the
  investigation
- All files were adapted to KiCad 7 format and many symbols and footprints
  were replaced with newer ones.
Parts:
- C10, C11, C12, C13, C14, C15, C16, C17, C5, C6, C7, C8, C9: symbol pspice:CAP -> Device:C
- J1: symbol Connector:Conn_01x02_Male -> Connector:Conn_01x02_Pin
Other:
- moved on the sheet: Y1
