File: connectors.kicad_sch (KiCad schematic)
At the start: 19 parts, among them J10 Serial, J11 Barrel_Jack_Switch, J12 Power, J13 RX In, J14 GND, J15 TX Out, J16 Port B, J2 Programming, J3 SHIFT0, J4 SHIFT1, J5 PSS, J6 1MHZ, J7 Reset F9T, J8 ANT_VCC, J9 F9T Connector

Commit message: Change to use 4 layers
- In1 is GND layer
- In2 is 3.3V layer
- Additionally, a few test points were added
Parts:
- removed J16: Port B, Connector_PinHeader_2.54mm:PinHeader_1x08_P2.54mm_Vertical, symbol Connector:Conn_01x08_Male
- added C31: 1u, Capacitor_SMD:C_1210_3225Metric, symbol Device:C
- added FB1: 33uH, Capacitor_SMD:C_0805_2012Metric, symbol Device:FerriteBead_Small
- added J16: Conn_01x09_Male, Connector_PinHeader_2.54mm:PinHeader_1x09_P2.54mm_Vertical, symbol Connector:Conn_01x09_Male
Connections:
- net B0: now also J16.1 (Pin_1)
- net B1: now also J16.2 (Pin_2)
- net B2: now also J16.3 (Pin_3)
- net B3: now also J16.4 (Pin_4)
- net B4: now also J16.5 (Pin_5)
- net B5: now also J16.6 (Pin_6)
- net B6: now also J16.7 (Pin_7)
- net B7: now also J16.8 (Pin_8)
- net GND: now also C31.2, J16.9 (Pin_9)
- net VCC_ANT: now also FB1.1; no longer J8.1 (Pin_1)
- new net: C31.1, FB1.2, J8.1 (Pin_1)
Other:
- moved on the sheet: C1, J8

Commit message: Fix inverse numbering of programming header
Connections:
- net +3.3V: now also J2.1 (Pin_1); no longer J2.4 (Pin_4)
- net GND: now also J2.4 (Pin_4); no longer J2.1 (Pin_1)
- net SWCLK: now also J2.3 (Pin_3); no longer J2.2 (Pin_2)
- net SWDIO: now also J2.2 (Pin_2); no longer J2.3 (Pin_3)
Other:
- moved on the sheet: J2

Commit message: Release board rev1
Ferrite bead 1 was removed (not needed)
Parts:
- removed FB1: 33uH, Capacitor_SMD:C_0805_2012Metric, symbol Device:FerriteBead_Small
Connections:
- net VCC_ANT: now also C31.1, J8.1 (Pin_1)
Changed lines of the file:
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@@
     (stroke (width 0) (type default) (color 0 0 0 0))
   )
-  (wire (pts (xy 110.49 97.79) (xy 114.3 97.79))
+  (wire (pts (xy 110.49 97.79) (xy 120.65 97.79))
     (stroke (width 0) (type default) (color 0 0 0 0))
   )
@@
   )
   (wire (pts (xy 60.96 142.24) (xy 92.71 142.24))
-    (stroke (width 0) (type default) (color 0 0 0 0))
-  )
-  (wire (pts (xy 119.38 97.79) (xy 120.65 97.79))
     (stroke (width 0) (type default) (color 0 0 0 0))
   )
@@
     (pin "1")
   )
-  (symbol (lib_id "Device:FerriteBead_Small") (at 116.84 97.79 90) (unit 1)
-    (in_bom yes) (on_board yes)
-    (property "Reference" "FB1" (id 0) (at 119.38 95.25 90))
-    (property "Value" "33uH" (id 1) (at 114.3 95.25 90))
-    (property "Footprint" "Capacitor_SMD:C_0805_2012Metric" (id 2) (at 116.84 99.568 90)
-      (effects (font (size 1.27 1.27)) hide)
-    )
-    (property "Datasheet" "~" (id 3) (at 116.84 97.79 0)
-      (effects (font (size 1.27 1.27)) hide)
-    )
-    (pin "1")
-    (pin "2")
-  )
   (symbol (lib_id "Connector:Conn_01x09_Male") (at 81.28 43.18 0) (unit 1)

Commit message: Add pull up resistors to SWD signals
Parts:
- added R4, R5: 10k, Resistor_SMD:R_0805_2012Metric, symbol Device:R
Connections:
- net +3.3V: now also R4.1, R5.1
- net SWCLK: now also R5.2
- net SWDIO: now also R4.2
Changed lines of the file:
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@@
   (junction (at 245.11 36.83) (diameter 0) (color 0 0 0 0)
   )
+  (junction (at 43.18 29.21) (diameter 0) (color 0 0 0 0)
+  )
   (junction (at 254 97.79) (diameter 0) (color 0 0 0 0)
   )
@@
   (junction (at 110.49 97.79) (diameter 0) (color 0 0 0 0)
   )
+  (junction (at 52.07 29.21) (diameter 0) (color 0 0 0 0)
+  )
   (junction (at 254 129.54) (diameter 0) (color 0 0 0 0)
   )
+  (junction (at 43.18 41.91) (diameter 0) (color 0 0 0 0)
+  )
   (junction (at 149.86 43.18) (diameter 0) (color 0 0 0 0)
   )
@@
   )
   (junction (at 254 21.59) (diameter 0) (color 0 0 0 0)
+  )
+  (junction (at 34.29 39.37) (diameter 0) (color 0 0 0 0)
   )
   (no_connect (at 104.14 163.83))
@@
     (stroke (width 0) (type default) (color 0 0 0 0))
   )
+  (wire (pts (xy 43.18 36.83) (xy 43.18 41.91))
+    (stroke (width 0) (type default) (color 0 0 0 0))
+  )
   (wire (pts (xy 92.71 142.24) (xy 92.71 152.4))
     (stroke (width 0) (type default) (color 0 0 0 0))
@@
     (stroke (width 0) (type default) (color 0 0 0 0))
   )
+  (wire (pts (xy 34.29 29.21) (xy 43.18 29.21))
+    (stroke (width 0) (type default) (color 0 0 0 0))
+  )
   (polyline (pts (xy 187.96 124.46) (xy 144.78 124.46))
     (stroke (width 0) (type default) (color 0 0 0 0))
   )
+  (wire (pts (xy 43.18 41.91) (xy 52.07 41.91))
+    (stroke (width 0) (type default) (color 0 0 0 0))
+  )
   (polyline (pts (xy 187.96 68.58) (xy 187.96 16.51))
     (stroke (width 0) (type default) (color 0 0 0 0))
@@
     (stroke (width 0) (type default) (color 0 0 0 0))
   )
+  (wire (pts (xy 34.29 39.37) (xy 52.07 39.37))
+    (stroke (width 0) (type default) (color 0 0 0 0))
+  )
   (polyline (pts (xy 114.3 16.51) (xy 114.3 68.58))
     (stroke (width 0) (type default) (color 0 0 0 0))
@@
     (stroke (width 0) (type default) (color 0 0 0 0))
   )
-  (wire (pts (xy 52.07 33.02) (xy 52.07 36.83))
+  (wire (pts (xy 52.07 29.21) (xy 52.07 36.83))
     (stroke (width 0) (type default) (color 0 0 0 0))
   )
@@
     (stroke (width 0) (type default) (color 0 0 0 0))
   )
+  (wire (pts (xy 43.18 29.21) (xy 52.07 29.21))
+    (stroke (width 0) (type default) (color 0 0 0 0))
+  )
   (wire (pts (xy 60.96 168.91) (xy 62.23 168.91))
     (stroke (width 0) (type default) (color 0 0 0 0))
   )
-  (wire (pts (xy 30.48 41.91) (xy 52.07 41.91))
+  (wire (pts (xy 30.48 41.91) (xy 43.18 41.91))
     (stroke (width 0) (type default) (color 0 0 0 0))
   )
@@
     (stroke (width 0) (type default) (color 0 0 0 0))
   )
+  (wire (pts (xy 34.29 36.83) (xy 34.29 39.37))
+    (stroke (width 0) (type default) (color 0 0 0 0))
+  )
   (wire (pts (xy 100.33 156.21) (xy 104.14 156.21))
     (stroke (width 0) (type default) (color 0 0 0 0))
@@
     (stroke (width 0) (type default) (color 0 0 0 0))
   )
-  (wire (pts (xy 30.48 39.37) (xy 52.07 39.37))
+  (wire (pts (xy 30.48 39.37) (xy 34.29 39.37))
     (stroke (width 0) (type default) (color 0 0 0 0))
   )
@@
     (pin "1")
   )
+  (symbol (lib_id "Device:R") (at 34.29 33.02 0) (unit 1)
+    (in_bom yes) (on_board yes) (fields_autoplaced)
+    (property "Reference" "R4" (id 0) (at 36.83 31.7499 0)
+      (effects (font (size 1.27 1.27)) (justify left))
+    )
+    (property "Value" "10k" (id 1) (at 36.83 34.2899 0)
+      (effects (font (size 1.27 1.27)) (justify left))
+    )
+    (property "Footprint" "Resistor_SMD:R_0805_2012Metric" (id 2) (at 32.512 33.02 90)
+      (effects (font (size 1.27 1.27)) hide)
+    )
+    (property "Datasheet" "~" (id 3) (at 34.29 33.02 0)
+      (effects (font (size 1.27 1.27)) hide)
+    )
+    (pin "1")
+    (pin "2")
+  )
   (symbol (lib_id "power:GND") (at 149.86 44.45 0) (unit 1)
     (in_bom yes) (on_board yes) (fields_autoplaced)
@@
     (pin "1")
   )
-  (symbol (lib_id "power:+3.3V") (at 52.07 33.02 0) (unit 1)
-    (in_bom yes) (on_board yes) (fields_autoplaced)
-    (property "Reference" "#PWR0136" (id 0) (at 52.07 36.83 0)
-      (effects (font (size 1.27 1.27)) hide)
-    )
-    (property "Value" "+3.3V" (id 1) (at 52.07 27.94 0))
-    (property "Footprint" "" (id 2) (at 52.07 33.02 0)
-      (effects (font (size 1.27 1.27)) hide)
-    )
-    (property "Datasheet" "" (id 3) (at 52.07 33.02 0)
+  (symbol (lib_id "power:+3.3V") (at 52.07 29.21 0) (unit 1)
+    (in_bom yes) (on_board yes) (fields_autoplaced)
+    (property "Reference" "#PWR0136" (id 0) (at 52.07 33.02 0)
+      (effects (font (size 1.27 1.27)) hide)
+    )
+    (property "Value" "+3.3V" (id 1) (at 52.07 24.13 0))
+    (property "Footprint" "" (id 2) (at 52.07 29.21 0)
+      (effects (font (size 1.27 1.27)) hide)
+    )
+    (property "Datasheet" "" (id 3) (at 52.07 29.21 0)
       (effects (font (size 1.27 1.27)) hide)
     )
@@
     (pin "5")
   )
+  (symbol (lib_id "Device:R") (at 43.18 33.02 0) (unit 1)
+    (in_bom yes) (on_board yes) (fields_autoplaced)
+    (property "Reference" "R5" (id 0) (at 45.72 31.7499 0)
+      (effects (font (size 1.27 1.27)) (justify left))
+    )
+    (property "Value" "10k" (id 1) (at 45.72 34.2899 0)
+      (effects (font (size 1.27 1.27)) (justify left))
+    )
+    (property "Footprint" "Resistor_SMD:R_0805_2012Metric" (id 2) (at 41.402 33.02 90)
+      (effects (font (size 1.27 1.27)) hide)
+    )
+    (property "Datasheet" "~" (id 3) (at 43.18 33.02 0)
+      (effects (font (size 1.27 1.27)) hide)
+    )
+    (pin "1")
+    (pin "2")
+  )
   (symbol (lib_id "Connector:Conn_01x02_Male") (at 38.1 97.79 0) (unit 1)
