File: connectors.kicad_sch (KiCad schematic)
At the start: 22 parts, among them J10 Serial, J11 Barrel_Jack_Switch, J12 Power, J13 RX In, J14 GND, J15 TX Out, J16 Conn_01x09_Male, J2 Programming, J3 SHIFT0, J4 SHIFT1, J5 PSS, J6 1MHZ, J7 Reset F9T, J8 ANT_VCC, J9 F9T Connector

Commit message: Rev3: Fix GPS receiver start problem and update to KiCad 7
- Pin TP2 of GPS receiver seems to be pulled down briefly at start time,
  this triggers the safe boot mode. A buffer was added to address this
  issue. Thanks Chris C. for the fix and thanks Paul H. for the
  investigation
- All files were adapted to KiCad 7 format and many symbols and footprints
  were replaced with newer ones.
Parts:
- J13, J14, J15: symbol Connector:Conn_01x03_Male -> Connector:Conn_01x03_Pin
- J16: symbol Connector:Conn_01x09_Male -> Connector:Conn_01x09_Pin
- J2: symbol Connector:Conn_01x04_Male -> Connector:Conn_01x04_Pin
- J7, J8: symbol Connector:Conn_01x02_Male -> Connector:Conn_01x02_Pin
Changed lines of the file:
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@@
     (effects (font (size 1.27 1.27)) (justify right))
   )
-  (symbol (lib_id "Connector:Conn_01x03_Male") (at 55.88 168.91 0) (unit 1)
+  (symbol (lib_id "Connector:Conn_01x03_Pin") (at 55.88 168.91 0) (unit 1)
     (in_bom yes) (on_board yes) (dnp no)
     (property "Reference" "J15" (at 53.34 167.64 0)
@@
     )
   )
-  (symbol (lib_id "Connector:Conn_01x02_Male") (at 127 97.79 180) (unit 1)
+  (symbol (lib_id "Connector:Conn_01x02_Pin") (at 127 97.79 180) (unit 1)
     (in_bom yes) (on_board yes) (dnp no) (fields_autoplaced)
     (property "Reference" "J8" (at 128.27 95.2499 0)
@@
     )
   )
-  (symbol (lib_id "Connector:Conn_01x03_Male") (at 55.88 139.7 0) (unit 1)
+  (symbol (lib_id "Connector:Conn_01x03_Pin") (at 55.88 139.7 0) (unit 1)
     (in_bom yes) (on_board yes) (dnp no)
     (property "Reference" "J13" (at 52.07 137.16 0)
@@
     )
   )
-  (symbol (lib_id "Connector:Conn_01x04_Male") (at 57.15 39.37 0) (mirror y) (unit 1)
+  (symbol (lib_id "Connector:Conn_01x04_Pin") (at 57.15 39.37 0) (mirror y) (unit 1)
     (in_bom yes) (on_board yes) (dnp no)
     (property "Reference" "J2" (at 57.15 46.99 0)
@@
     )
   )
-  (symbol (lib_id "Connector:Conn_01x03_Male") (at 55.88 154.94 0) (unit 1)
+  (symbol (lib_id "Connector:Conn_01x03_Pin") (at 55.88 154.94 0) (unit 1)
     (in_bom yes) (on_board yes) (dnp no)
     (property "Reference" "J14" (at 54.61 153.67 0)
@@
     )
   )
-  (symbol (lib_id "Connector:Conn_01x09_Male") (at 81.28 43.18 0) (unit 1)
+  (symbol (lib_id "Connector:Conn_01x09_Pin") (at 81.28 43.18 0) (unit 1)
     (in_bom yes) (on_board yes) (dnp no) (fields_autoplaced)
     (property "Reference" "J16" (at 81.915 27.94 0)
@@
     )
   )
-  (symbol (lib_id "Connector:Conn_01x02_Male") (at 38.1 97.79 0) (unit 1)
+  (symbol (lib_id "Connector:Conn_01x02_Pin") (at 38.1 97.79 0) (unit 1)
     (in_bom yes) (on_board yes) (dnp no) (fields_autoplaced)
     (property "Reference" "J7" (at 38.735 92.71 0)
