File: power.kicad_sch (KiCad schematic)
At the start: 7 parts, among them U1 AMS1117

Commit message: Rev3: Fix GPS receiver start problem and update to KiCad 7
- Pin TP2 of GPS receiver seems to be pulled down briefly at start time,
  this triggers the safe boot mode. A buffer was added to address this
  issue. Thanks Chris C. for the fix and thanks Paul H. for the
  investigation
- All files were adapted to KiCad 7 format and many symbols and footprints
  were replaced with newer ones.
Parts:
- C29, C3, C30, C4: symbol pspice:CAP -> Device:C
Other:
- note added: "Max consumptions: - STM32 microcontroller 100mA at 3.3V - GPS antenna 100mA at 5V - GPS receiver 100mA at 3.3V - Level shifter 1 300mA at 5V - Level shifter 2 300mA at 5V Max Power Consumption ~4W"
- note removed: "Max consumptions: - STM32 microcontroller 100mA at 3.3V - GPS antenna 100mA at 5V - GPS receiver 100mA at 3.3V Max Power Consumption ~1.2W"
Changed lines of the file:
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@@
   (junction (at 73.66 86.36) (diameter 0) (color 0 0 0 0)
   )
-  (wire (pts (xy 73.66 83.82) (xy 73.66 86.36))
+  (wire (pts (xy 58.42 71.12) (xy 58.42 73.66))
+    (stroke (width 0) (type default))
+  )
+  (wire (pts (xy 73.66 81.28) (xy 73.66 86.36))
     (stroke (width 0) (type default))
   )
@@
     (stroke (width 0) (type default))
   )
-  (wire (pts (xy 130.81 83.82) (xy 130.81 86.36))
+  (wire (pts (xy 130.81 81.28) (xy 130.81 86.36))
     (stroke (width 0) (type default))
   )
@@
     (stroke (width 0) (type default))
   )
+  (wire (pts (xy 73.66 71.12) (xy 73.66 73.66))
+    (stroke (width 0) (type default))
+  )
   (wire (pts (xy 177.8 59.69) (xy 177.8 68.58))
     (stroke (width 0) (type default))
@@
     (stroke (width 0) (type default))
   )
-  (wire (pts (xy 58.42 83.82) (xy 58.42 86.36))
+  (wire (pts (xy 130.81 71.12) (xy 130.81 73.66))
+    (stroke (width 0) (type default))
+  )
+  (wire (pts (xy 101.6 71.12) (xy 101.6 73.66))
+    (stroke (width 0) (type default))
+  )
+  (wire (pts (xy 58.42 81.28) (xy 58.42 86.36))
     (stroke (width 0) (type default))
   )
@@
     (stroke (width 0) (type default))
   )
-  (wire (pts (xy 101.6 83.82) (xy 101.6 86.36))
-    (stroke (width 0) (type default))
-  )
-  (text "Max consumptions:\n- STM32 microcontroller 100mA at 3.3V\n- GPS antenna 100mA at 5V\n- GPS receiver 100mA at 3.3V\nMax Power Consumption ~1.2W"
+  (wire (pts (xy 101.6 81.28) (xy 101.6 86.36))
+    (stroke (width 0) (type default))
+  )
+  (text "Max consumptions:\n- STM32 microcontroller 100mA at 3.3V\n- GPS antenna 100mA at 5V\n- GPS receiver 100mA at 3.3V\n- Level shifter 1 300mA at 5V\n- Level shifter 2 300mA at 5V\nMax Power Consumption ~4W"
     (at 137.16 118.11 0)
     (effects (font (size 1.27 1.27)) (justify left bottom))
@@
     )
   )
-  (symbol (lib_id "pspice:CAP") (at 58.42 77.47 0) (unit 1)
+  (symbol (lib_id "Device:C") (at 58.42 77.47 0) (unit 1)
     (in_bom yes) (on_board yes) (dnp no) (fields_autoplaced)
     (property "Reference" "C29" (at 63.5 76.1999 0)
@@
       (effects (font (size 1.27 1.27)) (justify left))
     )
-    (property "Footprint" "Capacitor_SMD:C_1210_3225Metric" (at 58.42 77.47 0)
+    (property "Footprint" "Capacitor_SMD:C_1210_3225Metric" (at 59.3852 81.28 0)
       (effects (font (size 1.27 1.27)) hide)
     )
@@
     )
   )
-  (symbol (lib_id "pspice:CAP") (at 130.81 77.47 0) (unit 1)
+  (symbol (lib_id "Device:C") (at 130.81 77.47 0) (unit 1)
     (in_bom yes) (on_board yes) (dnp no) (fields_autoplaced)
     (property "Reference" "C30" (at 135.89 76.1999 0)
@@
       (effects (font (size 1.27 1.27)) (justify left))
     )
-    (property "Footprint" "Capacitor_SMD:C_1210_3225Metric" (at 130.81 77.47 0)
+    (property "Footprint" "Capacitor_SMD:C_1210_3225Metric" (at 131.7752 81.28 0)
       (effects (font (size 1.27 1.27)) hide)
     )
@@
     )
   )
-  (symbol (lib_id "pspice:CAP") (at 101.6 77.47 0) (unit 1)
+  (symbol (lib_id "Device:C") (at 101.6 77.47 0) (unit 1)
     (in_bom yes) (on_board yes) (dnp no) (fields_autoplaced)
     (property "Reference" "C4" (at 106.68 76.1999 0)
@@
       (effects (font (size 1.27 1.27)) (justify left))
     )
-    (property "Footprint" "Capacitor_SMD:C_1210_3225Metric" (at 101.6 77.47 0)
+    (property "Footprint" "Capacitor_SMD:C_1210_3225Metric" (at 102.5652 81.28 0)
       (effects (font (size 1.27 1.27)) hide)
     )
@@
     )
   )
-  (symbol (lib_id "pspice:CAP") (at 73.66 77.47 0) (unit 1)
+  (symbol (lib_id "Device:C") (at 73.66 77.47 0) (unit 1)
     (in_bom yes) (on_board yes) (dnp no) (fields_autoplaced)
     (property "Reference" "C3" (at 78.74 76.1999 0)
@@
       (effects (font (size 1.27 1.27)) (justify left))
     )
-    (property "Footprint" "Capacitor_SMD:C_1210_3225Metric" (at 73.66 77.47 0)
-      (effects (font (size 1.27 1.27)) hide)
-    )
+    (property "Footprint" "Capacitor_SMD:C_1210_3225Metric" (at 74.6252 81.28 0)
+      (effects (font (size 1.27 1.27)) hide)
+    )
