File: d2tsf-hw.kicad_sch (KiCad schematic)
At the start: 0 parts

Commit message: Add metadata to follow Diamond's standard and use a letter for the revision
Other:
- note added: "A (0) - Initial design"
- note added: "B - Fix wrong SWD wiring - Fix GPS receiver boot by adding a buffer (CC's contribution)"
- note added: "REVISIONS"
- company: Diamond Light Source -> Diamond Light Source LTD
Changed lines of the file:
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@@
     (title "D2TSF")
     (date "2022-10-27")
-    (rev "Rev2")
-    (company "Diamond Light Source")
+    (rev "B")
+    (company "Diamond Light Source LTD")
+    (comment 1 "DRG No: 1187445")
+    (comment 2 "CHK: AC")
+    (comment 3 "DRN: EPJ")
   )
   (wire (pts (xy 114.3 83.82) (xy 139.7 83.82))
@@
     (stroke (width 0) (type default))
   )
+  (rectangle (start 191.77 24.13) (end 276.86 151.13)
+    (stroke (width 0) (type dot))
+    (fill (type none))
+  )
+  (text "A (0)\n- Initial design" (at 195.58 36.83 0)
+    (effects (font (size 1.27 1.27)) (justify left bottom))
+  )
+  (text "B\n- Fix wrong SWD wiring\n- Fix GPS receiver boot by adding a buffer (CC's contribution)"
+    (at 195.58 46.99 0)
+    (effects (font (size 1.27 1.27)) (justify left bottom))
+  )
+  (text "REVISIONS" (at 195.58 27.94 0)
+    (effects (font (size 1.27 1.27)) (justify left bottom))
+  )
   (sheet (at 49.53 46.99) (size 48.26 27.94) (fields_autoplaced)
